File: Calma04/Calma04_hw/Calma04.sch (KiCad schematic (older format))
At the start: 49 parts, among them Q1 ALS-PT19-315C, SW1 SWITCH, SW2 BUTTON

Commit message: Calma04 sch renewed
Parts:
- D1: symbol D_SHOTTKY -> D_Shottky
- F1, F2: symbol FUSE0R -> Fuse0R
- HOLE2: symbol HOLE_METALLED -> HOLE_METALLED-RESCUE-Calma04
- Q1: symbol PHOTOTRANSISTOR -> Phototransistor
Changed lines of the file:
@@
 EESchema Schematic File Version 2
+LIBS:Calma04-rescue
 LIBS:Connectors_kl
 LIBS:pcb_details
@@
 LIBS:Transistors_kl
 LIBS:Calma04-cache
-EELAYER 27 0
+EELAYER 25 0
 EELAYER END
 $Descr A3 16535 11693
@@
 $EndComp
 $Comp
-L PHOTOTRANSISTOR Q1
+L Phototransistor Q1
 U 1 1 5102E147
 P 2050 2300
@@
 $EndComp
 $Comp
-L FUSE0R F1
+L Fuse0R F1
 U 1 1 518BEE94
 P 2500 8700
@@
 BAT_IN
 $Comp
-L HOLE_METALLED HOLE2
+L HOLE_METALLED-RESCUE-Calma04 HOLE2
 U 1 1 51E1095D
 P 13550 1600
@@
 $EndComp
 $Comp
-L FUSE0R F2
+L Fuse0R F2
 U 1 1 51E1315F
 P 4300 8050
@@
 $EndComp
 $Comp
-L D_SHOTTKY D1
+L D_Shottky D1
 U 1 1 51E13F5A
 P 9600 1500
